Commit message: #2 Robot Arm Position Fixed, README Updated.

File: rover_21_robotic_arm/arm_21_gazebo/urdf/arm_21_gazebo.urdf.xacro (robot description, xacro)
@@ -7,5 +7,5 @@
   <xacro:include filename="$(find rover_21_description)/urdf/rover_21_description.urdf.xacro" /> <!-- include rover base urdf as xacro-->
   <joint name="dummy" type="fixed"> <!-- dummy joint it is fixed joint that means it is not moveable this was joint that connet arm to rovers base-->
-    <origin xyz="0.25 0 0.15" rpy="0 0 0"/>
+    <origin xyz="0.15 0 0.12" rpy="0 0 0"/>
     <parent link="base_link"/>
     <child link="alt_plaka"/>

Commit message: #11 Change Camera Collision and Change PID gains.

File: rover_21_robotic_arm/arm_21_gazebo/urdf/arm_21_gazebo.urdf.xacro (robot description, xacro)
@@ -612,10 +612,10 @@
 <!-- 2 fpv camera pyhsicla propotions-->
 <link name="camera">
-  <collision>
+  <!-- <collision>
     <origin xyz="0 0 0" rpy="0 0 0" />
     <geometry>
       <box size="0.05 0.05 0.05" />
     </geometry>
-  </collision>
+  </collision> -->
   <visual>
     <origin xyz="0 0 0" rpy="0 0 0" />
@@ -625,10 +625,10 @@
     <material name="green" />
   </visual>
-  <inertial>
+  <!-- <inertial>
     <mass value="0.1" />
     <origin xyz="0 0 0" rpy="0 0 0" />
     <box_inertia m="0.1" x="0.05" y="0.05" z="0.05" />
     <inertia ixx="1e-6" ixy="0" ixz="0" iyy="1e-6" iyz="0" izz="1e-6" />
-  </inertial>
+  </inertial> -->
 </link>
 <joint name="camera_joint1" type="fixed">
@@ -639,10 +639,10 @@
 </joint>
 <link name="camera2">
-  <collision>
+  <!-- <collision>
     <origin xyz="0 0 0" rpy="0 0 0" />
     <geometry>
       <box size="0.05 0.05 0.05" />
     </geometry>
-  </collision>
+  </collision> -->
   <visual>
     <origin xyz="0 0 0" rpy="0 0 0" />
@@ -652,10 +652,10 @@
     <material name="green" />
   </visual>
-  <inertial>
+  <!-- <inertial>
     <mass value="0.1" />
     <origin xyz="0 0 0" rpy="0 0 0" />
     <box_inertia m="0.1" x="0.05" y="0.05" z="0.05" />
     <inertia ixx="1e-6" ixy="0" ixz="0" iyy="1e-6" iyz="0" izz="1e-6" />
-  </inertial>
+  </inertial> -->
 </link>
 <joint name="camera_joint2" type="fixed">

Commit message: #21 Robot Aerm Rover Mesh Changed.

File: rover_21_robotic_arm/arm_21_gazebo/urdf/arm_21_gazebo.urdf.xacro (robot description, xacro)
@@ -7,5 +7,5 @@
   <xacro:include filename="$(find rover_21_description)/urdf/rover_21_description.urdf.xacro" /> <!-- include rover base urdf as xacro-->
   <joint name="dummy" type="fixed"> <!-- dummy joint it is fixed joint that means it is not moveable this was joint that connet arm to rovers base-->
-    <origin xyz="0.15 0 0.12" rpy="0 0 0"/>
+    <origin xyz="0.34 0 0.14" rpy="0 0 0"/>
     <parent link="base_link"/>
     <child link="alt_plaka"/>

File: rover_21_robotic_arm/rover_21_description/urdf/rover_21_description.urdf.xacro (robot description, xacro)
@@ -26,22 +26,22 @@
       <origin
         xyz="0 0 0"
-        rpy="0 0 0" />
-      <geometry>
-        <mesh
-          filename="package://rover_21_description/meshes/base_link.STL" />
-      </geometry>
-      <material
-        name="">
-        <color
-          rgba="0.792156862745098 0.819607843137255 0.933333333333333 1" />
-      </material>
-    </visual>
-    <collision>
-      <origin
-        xyz="0 0 0"
-        rpy="0 0 0" />
-      <geometry>
-        <mesh
-          filename="package://rover_21_description/meshes/base_link.STL" />
+        rpy="0 0 -1.57" />
+      <geometry>
+        <mesh
+          filename="package://rover_21_description/meshes/base_link_new.stl"  scale="0.1 0.1 0.1"/>
+      </geometry>
+      <material
+        name="">
+        <color
+          rgba="0.792156862745098 0.819607843137255 0.933333333333333 1" />
+      </material>
+    </visual>
+    <collision>
+      <origin
+        xyz="0 0 0"
+        rpy="0 0 -1.57" />
+      <geometry>
+        <mesh
+          filename="package://rover_21_description/meshes/base_link_new.stl"  scale="0.1 0.1 0.1"/>
       </geometry>
     </collision>
@@ -69,19 +69,19 @@
       <geometry>
         <mesh
-          filename="package://rover_21_description/meshes/left_front_link.STL" />
-      </geometry>
-      <material
-        name="">
-        <color
-          rgba="0.792156862745098 0.819607843137255 0.933333333333333 1" />
-      </material>
-    </visual>
-    <collision>
-      <origin
-        xyz="0 0 0"
-        rpy="0 0 0" />
-      <geometry>
-        <mesh
-          filename="package://rover_21_description/meshes/left_front_link.STL" />
+          filename="package://rover_21_description/meshes/left_front.stl"  scale="0.1 0.1 0.1"/>
+      </geometry>
+      <material
+        name="">
+        <color
+          rgba="0.792156862745098 0.819607843137255 0.933333333333333 1" />
+      </material>
+    </visual>
+    <collision>
+      <origin
+        xyz="0 0 0"
+        rpy="0 0 0" />
+      <geometry>
+        <mesh
+          filename="package://rover_21_description/meshes/left_front.stl"  scale="0.1 0.1 0.1"/>
       </geometry>
     </collision>
@@ -122,19 +122,19 @@
       <geometry>
         <mesh
-          filename="package://rover_21_description/meshes/right_front_link.STL" />
-      </geometry>
-      <material
-        name="">
-        <color
-          rgba="0.792156862745098 0.819607843137255 0.933333333333333 1" />
-      </material>
-    </visual>
-    <collision>
-      <origin
-        xyz="0 0 0"
-        rpy="0 0 0" />
-      <geometry>
-        <mesh
-          filename="package://rover_21_description/meshes/right_front_link.STL" />
+          filename="package://rover_21_description/meshes/right_front.stl"  scale="0.1 0.1 0.1"/>
+      </geometry>
+      <material
+        name="">
+        <color
+          rgba="0.792156862745098 0.819607843137255 0.933333333333333 1" />
+      </material>
+    </visual>
+    <collision>
+      <origin
+        xyz="0 0 0"
+        rpy="0 0 0" />
+      <geometry>
+        <mesh
+          filename="package://rover_21_description/meshes/right_front.stl"  scale="0.1 0.1 0.1"/>
       </geometry>
     </collision>
@@ -175,19 +175,19 @@
       <geometry>
         <mesh
-          filename="package://rover_21_description/meshes/left_rear_link.STL" />
-      </geometry>
-      <material
-        name="">
-        <color
-          rgba="0.792156862745098 0.819607843137255 0.933333333333333 1" />
-      </material>
-    </visual>
-    <collision>
-      <origin
-        xyz="0 0 0"
-        rpy="0 0 0" />
-      <geometry>
-        <mesh
-          filename="package://rover_21_description/meshes/left_rear_link.STL" />
+          filename="package://rover_21_description/meshes/left_behind.stl"  scale="0.1 0.1 0.1"/>
+      </geometry>
+      <material
+        name="">
+        <color
+          rgba="0.792156862745098 0.819607843137255 0.933333333333333 1" />
+      </material>
+    </visual>
+    <collision>
+      <origin
+        xyz="0 0 0"
+        rpy="0 0 0" />
+      <geometry>
+        <mesh
+          filename="package://rover_21_description/meshes/left_behind.stl"  scale="0.1 0.1 0.1"/>
       </geometry>
     </collision>
@@ -228,19 +228,19 @@
       <geometry>
         <mesh
-          filename="package://rover_21_description/meshes/right_rear_link.STL" />
-      </geometry>
-      <material
-        name="">
-        <color
-          rgba="0.792156862745098 0.819607843137255 0.933333333333333 1" />
-      </material>
-    </visual>
-    <collision>
-      <origin
-        xyz="0 0 0"
-        rpy="0 0 0" />
-      <geometry>
-        <mesh
-          filename="package://rover_21_description/meshes/right_rear_link.STL" />
+          filename="package://rover_21_description/meshes/right_front.stl"  scale="0.1 0.1 0.1"/>
+      </geometry>
+      <material
+        name="">
+        <color
+          rgba="0.792156862745098 0.819607843137255 0.933333333333333 1" />
+      </material>
+    </visual>
+    <collision>
+      <origin
+        xyz="0 0 0"
+        rpy="0 0 0" />
+      <geometry>
+        <mesh
+          filename="package://rover_21_description/meshes/right_front.stl" scale="0.1 0.1 0.1"/>
       </geometry>
     </collision>
