Commit message: #36 Robot Arm 22 Position Controllers Added and Gazebo Actors Added.

File: rover_22_robotic_arm/arm_22_gazebo_pos/urdf/assembly.urdf.xacro (robot description, xacro)
@@ -1,7 +1,7 @@
 <?xml version="1.0" ?>
 <robot name="assembly" xmlns:xacro="http://www.ros.org/wiki/xacro">
-<xacro:include filename="$(find arm_22_gazebo)/urdf/materials.xacro" />
-<xacro:include filename="$(find arm_22_gazebo)/urdf/assembly.trans" />
-<xacro:include filename="$(find arm_22_gazebo)/urdf/assembly.gazebo" />
+<xacro:include filename="$(find arm_22_gazebo_pos)/urdf/materials.xacro" />
+<xacro:include filename="$(find arm_22_gazebo_pos)/urdf/assembly.trans" />
+<xacro:include filename="$(find arm_22_gazebo_pos)/urdf/assembly.gazebo" />
 <link name="world"> </link>
 <joint name="dummy_joint" type="fixed">
@@ -19,5 +19,5 @@
     <origin rpy="0 0 0" xyz="0 0 0"/>
     <geometry>
-      <mesh filename="package://arm_22_gazebo/meshes/base_link.stl" scale="0.001 0.001 0.001"/>
+      <mesh filename="package://arm_22_gazebo_pos/meshes/base_link.stl" scale="0.001 0.001 0.001"/>
     </geometry>
     <material name="silver"/>
@@ -26,5 +26,5 @@
     <origin rpy="0 0 0" xyz="0 0 0"/>
     <geometry>
-      <mesh filename="package://arm_22_gazebo/meshes/base_link.stl" scale="0.001 0.001 0.001"/>
+      <mesh filename="package://arm_22_gazebo_pos/meshes/base_link.stl" scale="0.001 0.001 0.001"/>
     </geometry>
   </collision>
@@ -39,5 +39,5 @@
     <origin rpy="0 0 0" xyz="-0.0 -0.0 -0.0535"/>
     <geometry>
-      <mesh filename="package://arm_22_gazebo/meshes/1_2_link_1.stl" scale="0.001 0.001 0.001"/>
+      <mesh filename="package://arm_22_gazebo_pos/meshes/1_2_link_1.stl" scale="0.001 0.001 0.001"/>
     </geometry>
     <material name="silver"/>
@@ -46,5 +46,5 @@
     <origin rpy="0 0 0" xyz="-0.0 -0.0 -0.0535"/>
     <geometry>
-      <mesh filename="package://arm_22_gazebo/meshes/1_2_link_1.stl" scale="0.001 0.001 0.001"/>
+      <mesh filename="package://arm_22_gazebo_pos/meshes/1_2_link_1.stl" scale="0.001 0.001 0.001"/>
     </geometry>
   </collision>
@@ -59,5 +59,5 @@
     <origin rpy="0 0 0" xyz="-0.0215 -0.0 -0.141"/>
     <geometry>
-      <mesh filename="package://arm_22_gazebo/meshes/2_3_link_1.stl" scale="0.001 0.001 0.001"/>
+      <mesh filename="package://arm_22_gazebo_pos/meshes/2_3_link_1.stl" scale="0.001 0.001 0.001"/>
     </geometry>
     <material name="silver"/>
@@ -66,5 +66,5 @@
     <origin rpy="0 0 0" xyz="-0.0215 -0.0 -0.141"/>
     <geometry>
-      <mesh filename="package://arm_22_gazebo/meshes/2_3_link_1.stl" scale="0.001 0.001 0.001"/>
+      <mesh filename="package://arm_22_gazebo_pos/meshes/2_3_link_1.stl" scale="0.001 0.001 0.001"/>
     </geometry>
   </collision>
@@ -79,5 +79,5 @@
     <origin rpy="0 0 0" xyz="0.025 -0.0 -0.7965"/>
     <geometry>
-      <mesh filename="package://arm_22_gazebo/meshes/3_4_link_1.stl" scale="0.001 0.001 0.001"/>
+      <mesh filename="package://arm_22_gazebo_pos/meshes/3_4_link_1.stl" scale="0.001 0.001 0.001"/>
     </geometry>
     <material name="silver"/>
@@ -86,5 +86,5 @@
     <origin rpy="0 0 0" xyz="0.025 -0.0 -0.7965"/>
     <geometry>
-      <mesh filename="package://arm_22_gazebo/meshes/3_4_link_1.stl" scale="0.001 0.001 0.001"/>
+      <mesh filename="package://arm_22_gazebo_pos/meshes/3_4_link_1.stl" scale="0.001 0.001 0.001"/>
     </geometry>
   </collision>
@@ -99,5 +99,5 @@
     <origin rpy="0 0 0" xyz="-0.0 0.14925 -0.7965"/>
     <geometry>
-      <mesh filename="package://arm_22_gazebo/meshes/4_5_link_1.stl" scale="0.001 0.001 0.001"/>
+      <mesh filename="package://arm_22_gazebo_pos/meshes/4_5_link_1.stl" scale="0.001 0.001 0.001"/>
     </geometry>
     <material name="silver"/>
@@ -106,5 +106,5 @@
     <origin rpy="0 0 0" xyz="-0.0 0.14925 -0.7965"/>
     <geometry>
-      <mesh filename="package://arm_22_gazebo/meshes/4_5_link_1.stl" scale="0.001 0.001 0.001"/>
+      <mesh filename="package://arm_22_gazebo_pos/meshes/4_5_link_1.stl" scale="0.001 0.001 0.001"/>
     </geometry>
   </collision>
@@ -119,5 +119,5 @@
     <origin rpy="0 0 0" xyz="-0.055 0.54725 -0.7965"/>
     <geometry>
-      <mesh filename="package://arm_22_gazebo/meshes/5_6_link_1.stl" scale="0.001 0.001 0.001"/>
+      <mesh filename="package://arm_22_gazebo_pos/meshes/5_6_link_1.stl" scale="0.001 0.001 0.001"/>
     </geometry>
     <material name="silver"/>
@@ -126,5 +126,5 @@
     <origin rpy="0 0 0" xyz="-0.055 0.54725 -0.7965"/>
     <geometry>
-      <mesh filename="package://arm_22_gazebo/meshes/5_6_link_1.stl" scale="0.001 0.001 0.001"/>
+      <mesh filename="package://arm_22_gazebo_pos/meshes/5_6_link_1.stl" scale="0.001 0.001 0.001"/>
     </geometry>
   </collision>
@@ -139,5 +139,5 @@
     <origin rpy="0 0 0" xyz="-0.0 0.56925 -0.7965"/>
     <geometry>
-      <mesh filename="package://arm_22_gazebo/meshes/gripper_link_1.stl" scale="0.001 0.001 0.001"/>
+      <mesh filename="package://arm_22_gazebo_pos/meshes/gripper_link_1.stl" scale="0.001 0.001 0.001"/>
     </geometry>
     <material name="silver"/>
@@ -146,5 +146,5 @@
     <origin rpy="0 0 0" xyz="-0.0 0.56925 -0.7965"/>
     <geometry>
-      <mesh filename="package://arm_22_gazebo/meshes/gripper_link_1.stl" scale="0.001 0.001 0.001"/>
+      <mesh filename="package://arm_22_gazebo_pos/meshes/gripper_link_1.stl" scale="0.001 0.001 0.001"/>
     </geometry>
   </collision>
@@ -159,5 +159,5 @@
     <origin rpy="0 0 0" xyz="0.008 0.65425 -0.8115"/>
     <geometry>
-      <mesh filename="package://arm_22_gazebo/meshes/parmak_1_link_1.stl" scale="0.001 0.001 0.001"/>
+      <mesh filename="package://arm_22_gazebo_pos/meshes/parmak_1_link_1.stl" scale="0.001 0.001 0.001"/>
     </geometry>
     <material name="silver"/>
@@ -166,5 +166,5 @@
     <origin rpy="0 0 0" xyz="0.008 0.65425 -0.8115"/>
     <geometry>
-      <mesh filename="package://arm_22_gazebo/meshes/parmak_1_link_1.stl" scale="0.001 0.001 0.001"/>
+      <mesh filename="package://arm_22_gazebo_pos/meshes/parmak_1_link_1.stl" scale="0.001 0.001 0.001"/>
     </geometry>
   </collision>
@@ -179,5 +179,5 @@
     <origin rpy="0 0 0" xyz="-0.008 0.65425 -0.8115"/>
     <geometry>
-      <mesh filename="package://arm_22_gazebo/meshes/parmak_2_link_1.stl" scale="0.001 0.001 0.001"/>
+      <mesh filename="package://arm_22_gazebo_pos/meshes/parmak_2_link_1.stl" scale="0.001 0.001 0.001"/>
     </geometry>
     <material name="silver"/>
@@ -186,5 +186,5 @@
     <origin rpy="0 0 0" xyz="-0.008 0.65425 -0.8115"/>
     <geometry>
-      <mesh filename="package://arm_22_gazebo/meshes/parmak_2_link_1.stl" scale="0.001 0.001 0.001"/>
+      <mesh filename="package://arm_22_gazebo_pos/meshes/parmak_2_link_1.stl" scale="0.001 0.001 0.001"/>
     </geometry>
   </collision>
