Commit message: #19 Change Robot Arm Rover.

File: rover_21_robotic_arm/rover_21_description/urdf/rover_21_description.urdf.xacro (robot description, xacro)
@@ -5,7 +5,6 @@
 <robot
   name="rover_21_description" xmlns:xacro="http://www.ros.org/wiki/xacro">
-  <!--xacro:include filename="$(find rover_21_description)/urdf/vlp16.urdf.xacro"/>
-  <xacro:property name="cameraSize" value="0.05"/>
-  <xacro:property name="cameraMass" value="0.1"/-->
+  <!-- <xacro:property name="cameraSize" value="0.05"/>
+  <xacro:property name="cameraMass" value="0.1"/> -->
   <link
     name="base_link">
@@ -335,5 +334,5 @@
     </plugin>
   </gazebo-->
-   <gazebo>
+   <!-- <gazebo>
     <plugin name="imu_controller" filename="libhector_gazebo_ros_imu.so">
       <updateRate>30.0</updateRate>
@@ -361,5 +360,5 @@
       <drift>0.0001 0.0001 0.0001</drift>
     </plugin>
-  </gazebo>
+  </gazebo> -->
   <!--gazebo reference="camera">
      <sensor type="camera" name="camera">

Commit message: #48 Fixed files.

File: rover_21_robotic_arm/rover_21_description/urdf/rover_21_description.urdf.xacro (robot description, xacro)
@@ -5,6 +5,6 @@
 <robot
   name="rover_21_description" xmlns:xacro="http://www.ros.org/wiki/xacro">
-  <!-- <xacro:property name="cameraSize" value="0.05"/>
-  <xacro:property name="cameraMass" value="0.1"/> -->
+  <xacro:property name="cameraSize" value="0.05"/>
+  <xacro:property name="cameraMass" value="0.1"/>
   <link
     name="base_link">
