Commit message: #51 New link lenghts.

File: rover_22_robotic_arm/new_links/arm_22_gazebo_pos_55_55/urdf/assembly.urdf.xacro (robot description, xacro)
@@ -2,7 +2,7 @@
 <robot name="assembly"
   xmlns:xacro="http://www.ros.org/wiki/xacro">
-  <xacro:include filename="$(find arm_22_gazebo_pos)/urdf/materials.xacro" />
-  <xacro:include filename="$(find arm_22_gazebo_pos)/urdf/assembly.trans" />
-  <xacro:include filename="$(find arm_22_gazebo_pos)/urdf/assembly.gazebo" />
+  <xacro:include filename="$(find arm_22_gazebo_pos_55_55)/urdf/materials.xacro" />
+  <xacro:include filename="$(find arm_22_gazebo_pos_55_55)/urdf/assembly.trans" />
+  <xacro:include filename="$(find arm_22_gazebo_pos_55_55)/urdf/assembly.gazebo" />
   <link name="world"></link>
   <joint name="dummy_joint" type="fixed">
@@ -20,5 +20,5 @@
       <origin rpy="0 0 0" xyz="0 0 0"/>
       <geometry>
-        <mesh filename="package://arm_22_gazebo_pos/meshes/base_link.stl" scale="0.001 0.001 0.001"/>
+        <mesh filename="package://arm_22_gazebo_pos_55_55/meshes/base_link.stl" scale="0.001 0.001 0.001"/>
       </geometry>
       <material name="silver"/>
@@ -27,5 +27,5 @@
       <origin rpy="0 0 0" xyz="0 0 0"/>
       <geometry>
-        <mesh filename="package://arm_22_gazebo_pos/meshes/base_link.stl" scale="0.001 0.001 0.001"/>
+        <mesh filename="package://arm_22_gazebo_pos_55_55/meshes/base_link.stl" scale="0.001 0.001 0.001"/>
       </geometry>
     </collision>
@@ -40,5 +40,5 @@
       <origin rpy="0 0 0" xyz="-0.0 -0.0 -0.0535"/>
       <geometry>
-        <mesh filename="package://arm_22_gazebo_pos/meshes/1_2_link_1.stl" scale="0.001 0.001 0.001"/>
+        <mesh filename="package://arm_22_gazebo_pos_55_55/meshes/1_2_link_1.stl" scale="0.001 0.001 0.001"/>
       </geometry>
       <material name="silver"/>
@@ -47,5 +47,5 @@
       <origin rpy="0 0 0" xyz="-0.0 -0.0 -0.0535"/>
       <geometry>
-        <mesh filename="package://arm_22_gazebo_pos/meshes/1_2_link_1.stl" scale="0.001 0.001 0.001"/>
+        <mesh filename="package://arm_22_gazebo_pos_55_55/meshes/1_2_link_1.stl" scale="0.001 0.001 0.001"/>
       </geometry>
     </collision>
@@ -58,14 +58,16 @@
     </inertial>
     <visual>
-      <origin rpy="0 0 0" xyz="-0.0215 -0.0 -0.141"/>
-      <geometry>
-        <mesh filename="package://arm_22_gazebo_pos/meshes/2_3_link_1.stl" scale="0.001 0.001 0.001"/>
-      </geometry>
-      <material name="silver"/>
-    </visual>
-    <collision>
-      <origin rpy="0 0 0" xyz="-0.0215 -0.0 -0.141"/>
-      <geometry>
-        <mesh filename="package://arm_22_gazebo_pos/meshes/2_3_link_1.stl" scale="0.001 0.001 0.001"/>
+      <origin rpy="-1.57 0 0" xyz="-0.0 0.0 0.3"/>
+      <geometry>
+        <!-- <mesh filename="package://arm_22_gazebo_pos_55_55/meshes/2_3_link_1.stl" scale="0.001 0.001 0.001"/> -->
+        <box size=" 0.05 0.55 0.05" />
+      </geometry>
+      <material name="silver"/>
+    </visual>
+    <collision>
+      <origin rpy="-1.57 0 0" xyz="-0.0 -0.0 0.3"/>
+      <geometry>
+        <!-- <mesh filename="package://arm_22_gazebo_pos_55_55/meshes/2_3_link_1.stl" scale="0.001 0.001 0.001"/> -->
+        <box size="0.05 0.55 0.05" />
       </geometry>
     </collision>
@@ -78,14 +80,16 @@
     </inertial>
     <visual>
-      <origin rpy="0 0 0" xyz="0.025 -0.0 -0.7965"/>
-      <geometry>
-        <mesh filename="package://arm_22_gazebo_pos/meshes/3_4_link_1.stl" scale="0.001 0.001 0.001"/>
-      </geometry>
-      <material name="silver"/>
-    </visual>
-    <collision>
-      <origin rpy="0 0 0" xyz="0.025 -0.0 -0.7965"/>
-      <geometry>
-        <mesh filename="package://arm_22_gazebo_pos/meshes/3_4_link_1.stl" scale="0.001 0.001 0.001"/>
+      <origin rpy="0 0 0" xyz="0.025 -0.14 -0.1"/>
+      <geometry>
+        <!-- <mesh filename="package://arm_22_gazebo_pos_55_55/meshes/3_4_link_1.stl" scale="0.001 0.001 0.001"/> -->
+        <box size="0.05 0.275 0.05" />
+      </geometry>
+      <material name="silver"/>
+    </visual>
+    <collision>
+      <origin rpy="0 0 0" xyz="0.025 -0.14 -0.1"/>
+      <geometry>
+        <!-- <mesh filename="package://arm_22_gazebo_pos_55_55/meshes/3_4_link_1.stl" scale="0.001 0.001 0.001"/> -->
+        <box size="0.05 0.275 0.05" />
       </geometry>
     </collision>
@@ -98,14 +102,16 @@
     </inertial>
     <visual>
-      <origin rpy="0 0 0" xyz="-0.0 0.14925 -0.7965"/>
-      <geometry>
-        <mesh filename="package://arm_22_gazebo_pos/meshes/4_5_link_1.stl" scale="0.001 0.001 0.001"/>
-      </geometry>
-      <material name="silver"/>
-    </visual>
-    <collision>
-      <origin rpy="0 0 0" xyz="-0.0 0.14925 -0.7965"/>
-      <geometry>
-        <mesh filename="package://arm_22_gazebo_pos/meshes/4_5_link_1.stl" scale="0.001 0.001 0.001"/>
+      <origin rpy="0 0 0" xyz="-0.0 -0.28325 -0.1"/>
+      <geometry>
+        <!-- <mesh filename="package://arm_22_gazebo_pos_55_55/meshes/4_5_link_1.stl" scale="0.001 0.001 0.001"/> -->
+        <box size="0.05 0.275 0.05" />
+      </geometry>
+      <material name="silver"/>
+    </visual>
+    <collision>
+      <origin rpy="0 0 0" xyz="-0.0 -0.283925 -0.1"/>
+      <geometry>
+        <!-- <mesh filename="package://arm_22_gazebo_pos_55_55/meshes/4_5_link_1.stl" scale="0.001 0.001 0.001"/> -->
+        <box size="0.05 0.275 0.05" />
       </geometry>
     </collision>
@@ -118,14 +124,14 @@
     </inertial>
     <visual>
-      <origin rpy="0 0 0" xyz="-0.055 0.54725 -0.7965"/>
-      <geometry>
-        <mesh filename="package://arm_22_gazebo_pos/meshes/5_6_link_1.stl" scale="0.001 0.001 0.001"/>
-      </geometry>
-      <material name="silver"/>
-    </visual>
-    <collision>
-      <origin rpy="0 0 0" xyz="-0.055 0.54725 -0.7965"/>
-      <geometry>
-        <mesh filename="package://arm_22_gazebo_pos/meshes/5_6_link_1.stl" scale="0.001 0.001 0.001"/>
+      <origin rpy="0 0 0" xyz="-0.055 0.44725 -0.8965"/>
+      <geometry>
+        <mesh filename="package://arm_22_gazebo_pos_55_55/meshes/5_6_link_1.stl" scale="0.001 0.001 0.001"/>
+      </geometry>
+      <material name="silver"/>
+    </visual>
+    <collision>
+      <origin rpy="0 0 0" xyz="-0.055 0.44725 -0.8965"/>
+      <geometry>
+        <mesh filename="package://arm_22_gazebo_pos_55_55/meshes/5_6_link_1.stl" scale="0.001 0.001 0.001"/>
       </geometry>
     </collision>
@@ -138,14 +144,14 @@
     </inertial>
     <visual>
-      <origin rpy="0 0 0" xyz="-0.0 0.56925 -0.7965"/>
-      <geometry>
-        <mesh filename="package://arm_22_gazebo_pos/meshes/gripper_link_1.stl" scale="0.001 0.001 0.001"/>
-      </geometry>
-      <material name="silver"/>
-    </visual>
-    <collision>
-      <origin rpy="0 0 0" xyz="-0.0 0.56925 -0.7965"/>
-      <geometry>
-        <mesh filename="package://arm_22_gazebo_pos/meshes/gripper_link_1.stl" scale="0.001 0.001 0.001"/>
+      <origin rpy="0 0 0" xyz="-0.0 0.40925 -0.8965"/>
+      <geometry>
+        <mesh filename="package://arm_22_gazebo_pos_55_55/meshes/gripper_link_1.stl" scale="0.001 0.001 0.001"/>
+      </geometry>
+      <material name="silver"/>
+    </visual>
+    <collision>
+      <origin rpy="0 0 0" xyz="-0.0 0.40925 -0.8965"/>
+      <geometry>
+        <mesh filename="package://arm_22_gazebo_pos_55_55/meshes/gripper_link_1.stl" scale="0.001 0.001 0.001"/>
       </geometry>
     </collision>
@@ -158,14 +164,14 @@
     </inertial>
     <visual>
-      <origin rpy="0 0 0" xyz="0.008 0.65425 -0.8115"/>
-      <geometry>
-        <mesh filename="package://arm_22_gazebo_pos/meshes/parmak_1_link_1.stl" scale="0.001 0.001 0.001"/>
-      </geometry>
-      <material name="silver"/>
-    </visual>
-    <collision>
-      <origin rpy="0 0 0" xyz="0.008 0.65425 -0.8115"/>
-      <geometry>
-        <mesh filename="package://arm_22_gazebo_pos/meshes/parmak_1_link_1.stl" scale="0.001 0.001 0.001"/>
+      <origin rpy="0 0 0" xyz="0.008 0.4925 -0.9115"/>
+      <geometry>
+        <mesh filename="package://arm_22_gazebo_pos_55_55/meshes/parmak_1_link_1.stl" scale="0.001 0.001 0.001"/>
+      </geometry>
+      <material name="silver"/>
+    </visual>
+    <collision>
+      <origin rpy="0 0 0" xyz="0.008 0.4925 -0.9115"/>
+      <geometry>
+        <mesh filename="package://arm_22_gazebo_pos_55_55/meshes/parmak_1_link_1.stl" scale="0.001 0.001 0.001"/>
       </geometry>
     </collision>
@@ -178,14 +184,14 @@
     </inertial>
     <visual>
-      <origin rpy="0 0 0" xyz="-0.008 0.65425 -0.8115"/>
-      <geometry>
-        <mesh filename="package://arm_22_gazebo_pos/meshes/parmak_2_link_1.stl" scale="0.001 0.001 0.001"/>
-      </geometry>
-      <material name="silver"/>
-    </visual>
-    <collision>
-      <origin rpy="0 0 0" xyz="-0.008 0.65425 -0.8115"/>
-      <geometry>
-        <mesh filename="package://arm_22_gazebo_pos/meshes/parmak_2_link_1.stl" scale="0.001 0.001 0.001"/>
+      <origin rpy="0 0 0" xyz="-0.008 0.49425 -0.9115"/>
+      <geometry>
+        <mesh filename="package://arm_22_gazebo_pos_55_55/meshes/parmak_2_link_1.stl" scale="0.001 0.001 0.001"/>
+      </geometry>
+      <material name="silver"/>
+    </visual>
+    <collision>
+      <origin rpy="0 0 0" xyz="-0.008 0.49425 -0.9115"/>
+      <geometry>
+        <mesh filename="package://arm_22_gazebo_pos_55_55/meshes/parmak_2_link_1.stl" scale="0.001 0.001 0.001"/>
       </geometry>
     </collision>

File: rover_22_robotic_arm/new_links/arm_22_gazebo_pos_65_67/urdf/assembly.urdf.xacro (robot description, xacro)
@@ -2,7 +2,7 @@
 <robot name="assembly"
   xmlns:xacro="http://www.ros.org/wiki/xacro">
-  <xacro:include filename="$(find arm_22_gazebo_pos)/urdf/materials.xacro" />
-  <xacro:include filename="$(find arm_22_gazebo_pos)/urdf/assembly.trans" />
-  <xacro:include filename="$(find arm_22_gazebo_pos)/urdf/assembly.gazebo" />
+  <xacro:include filename="$(find arm_22_gazebo_pos_65_67)/urdf/materials.xacro" />
+  <xacro:include filename="$(find arm_22_gazebo_pos_65_67)/urdf/assembly.trans" />
+  <xacro:include filename="$(find arm_22_gazebo_pos_65_67)/urdf/assembly.gazebo" />
   <link name="world"></link>
   <joint name="dummy_joint" type="fixed">
@@ -20,5 +20,5 @@
       <origin rpy="0 0 0" xyz="0 0 0"/>
       <geometry>
-        <mesh filename="package://arm_22_gazebo_pos/meshes/base_link.stl" scale="0.001 0.001 0.001"/>
+        <mesh filename="package://arm_22_gazebo_pos_65_67/meshes/base_link.stl" scale="0.001 0.001 0.001"/>
       </geometry>
       <material name="silver"/>
@@ -27,5 +27,5 @@
       <origin rpy="0 0 0" xyz="0 0 0"/>
       <geometry>
-        <mesh filename="package://arm_22_gazebo_pos/meshes/base_link.stl" scale="0.001 0.001 0.001"/>
+        <mesh filename="package://arm_22_gazebo_pos_65_67/meshes/base_link.stl" scale="0.001 0.001 0.001"/>
       </geometry>
     </collision>
@@ -40,5 +40,5 @@
       <origin rpy="0 0 0" xyz="-0.0 -0.0 -0.0535"/>
       <geometry>
-        <mesh filename="package://arm_22_gazebo_pos/meshes/1_2_link_1.stl" scale="0.001 0.001 0.001"/>
+        <mesh filename="package://arm_22_gazebo_pos_65_67/meshes/1_2_link_1.stl" scale="0.001 0.001 0.001"/>
       </geometry>
       <material name="silver"/>
@@ -47,5 +47,5 @@
       <origin rpy="0 0 0" xyz="-0.0 -0.0 -0.0535"/>
       <geometry>
-        <mesh filename="package://arm_22_gazebo_pos/meshes/1_2_link_1.stl" scale="0.001 0.001 0.001"/>
+        <mesh filename="package://arm_22_gazebo_pos_65_67/meshes/1_2_link_1.stl" scale="0.001 0.001 0.001"/>
       </geometry>
     </collision>
@@ -58,14 +58,16 @@
     </inertial>
     <visual>
-      <origin rpy="0 0 0" xyz="-0.0215 -0.0 -0.141"/>
-      <geometry>
-        <mesh filename="package://arm_22_gazebo_pos/meshes/2_3_link_1.stl" scale="0.001 0.001 0.001"/>
-      </geometry>
-      <material name="silver"/>
-    </visual>
-    <collision>
-      <origin rpy="0 0 0" xyz="-0.0215 -0.0 -0.141"/>
-      <geometry>
-        <mesh filename="package://arm_22_gazebo_pos/meshes/2_3_link_1.stl" scale="0.001 0.001 0.001"/>
+      <origin rpy="-1.57 0 0" xyz="-0.0 -0.0 0.3"/>
+      <geometry>
+        <!-- <mesh filename="package://arm_22_gazebo_pos_65_67/meshes/2_3_link_1.stl" scale="0.001 0.001 0.001"/> -->
+        <box size=" 0.05 0.65 0.05" />
+      </geometry>
+      <material name="silver"/>
+    </visual>
+    <collision>
+      <origin rpy="-1.57 0 0" xyz="-0.0 -0.0 0.3"/>
+      <geometry>
+        <!-- <mesh filename="package://arm_22_gazebo_pos_65_67/meshes/2_3_link_1.stl" scale="0.001 0.001 0.001"/> -->
+        <box size="0.05 0.65 0.05" />
       </geometry>
     </collision>
@@ -78,14 +80,16 @@
     </inertial>
     <visual>
-      <origin rpy="0 0 0" xyz="0.025 -0.0 -0.7965"/>
-      <geometry>
-        <mesh filename="package://arm_22_gazebo_pos/meshes/3_4_link_1.stl" scale="0.001 0.001 0.001"/>
-      </geometry>
-      <material name="silver"/>
-    </visual>
-    <collision>
-      <origin rpy="0 0 0" xyz="0.025 -0.0 -0.7965"/>
-      <geometry>
-        <mesh filename="package://arm_22_gazebo_pos/meshes/3_4_link_1.stl" scale="0.001 0.001 0.001"/>
+      <origin rpy="0 0 0" xyz="0.025 -0.15 -0.0"/>
+      <geometry>
+        <!-- <mesh filename="package://arm_22_gazebo_pos_65_67/meshes/3_4_link_1.stl" scale="0.001 0.001 0.001"/> -->
+        <box size="0.05 0.300 0.05" />
+      </geometry>
+      <material name="silver"/>
+    </visual>
+    <collision>
+      <origin rpy="0 0 0" xyz="0.025 -0.15 -0.0"/>
+      <geometry>
+        <!-- <mesh filename="package://arm_22_gazebo_pos_65_67/meshes/3_4_link_1.stl" scale="0.001 0.001 0.001"/> -->
+        <box size="0.05 0.300 0.05" />
       </geometry>
     </collision>
@@ -98,14 +102,16 @@
     </inertial>
     <visual>
-      <origin rpy="0 0 0" xyz="-0.0 0.14925 -0.7965"/>
-      <geometry>
-        <mesh filename="package://arm_22_gazebo_pos/meshes/4_5_link_1.stl" scale="0.001 0.001 0.001"/>
-      </geometry>
-      <material name="silver"/>
-    </visual>
-    <collision>
-      <origin rpy="0 0 0" xyz="-0.0 0.14925 -0.7965"/>
-      <geometry>
-        <mesh filename="package://arm_22_gazebo_pos/meshes/4_5_link_1.stl" scale="0.001 0.001 0.001"/>
+      <origin rpy="0 0 0" xyz="-0.0 -0.29925 -0.0"/>
+      <geometry>
+        <!-- <mesh filename="package://arm_22_gazebo_pos_65_67/meshes/4_5_link_1.stl" scale="0.001 0.001 0.001"/> -->
+        <box size="0.05 0.373 0.05" />
+      </geometry>
+      <material name="silver"/>
+    </visual>
+    <collision>
+      <origin rpy="0 0 0" xyz="-0.0 -0.29925 -0.0"/>
+      <geometry>
+        <!-- <mesh filename="package://arm_22_gazebo_pos_65_67/meshes/4_5_link_1.stl" scale="0.001 0.001 0.001"/> -->
+        <box size="0.05 0.373 0.05" />
       </geometry>
     </collision>
@@ -118,14 +124,14 @@
     </inertial>
     <visual>
-      <origin rpy="0 0 0" xyz="-0.055 0.54725 -0.7965"/>
-      <geometry>
-        <mesh filename="package://arm_22_gazebo_pos/meshes/5_6_link_1.stl" scale="0.001 0.001 0.001"/>
-      </geometry>
-      <material name="silver"/>
-    </visual>
-    <collision>
-      <origin rpy="0 0 0" xyz="-0.055 0.54725 -0.7965"/>
-      <geometry>
-        <mesh filename="package://arm_22_gazebo_pos/meshes/5_6_link_1.stl" scale="0.001 0.001 0.001"/>
+      <origin rpy="0 0 0" xyz="-0.055 0.39725 -0.7965"/>
+      <geometry>
+        <mesh filename="package://arm_22_gazebo_pos_65_67/meshes/5_6_link_1.stl" scale="0.001 0.001 0.001"/>
+      </geometry>
+      <material name="silver"/>
+    </visual>
+    <collision>
+      <origin rpy="0 0 0" xyz="-0.055 0.39725 -0.7965"/>
+      <geometry>
+        <mesh filename="package://arm_22_gazebo_pos_65_67/meshes/5_6_link_1.stl" scale="0.001 0.001 0.001"/>
       </geometry>
     </collision>
@@ -138,14 +144,14 @@
     </inertial>
     <visual>
-      <origin rpy="0 0 0" xyz="-0.0 0.56925 -0.7965"/>
-      <geometry>
-        <mesh filename="package://arm_22_gazebo_pos/meshes/gripper_link_1.stl" scale="0.001 0.001 0.001"/>
-      </geometry>
-      <material name="silver"/>
-    </visual>
-    <collision>
-      <origin rpy="0 0 0" xyz="-0.0 0.56925 -0.7965"/>
-      <geometry>
-        <mesh filename="package://arm_22_gazebo_pos/meshes/gripper_link_1.stl" scale="0.001 0.001 0.001"/>
+      <origin rpy="0 0 0" xyz="-0.0 0.41925 -0.7965"/>
+      <geometry>
+        <mesh filename="package://arm_22_gazebo_pos_65_67/meshes/gripper_link_1.stl" scale="0.001 0.001 0.001"/>
+      </geometry>
+      <material name="silver"/>
+    </visual>
+    <collision>
+      <origin rpy="0 0 0" xyz="-0.0 0.41925 -0.7965"/>
+      <geometry>
+        <mesh filename="package://arm_22_gazebo_pos_65_67/meshes/gripper_link_1.stl" scale="0.001 0.001 0.001"/>
       </geometry>
     </collision>
@@ -158,14 +164,14 @@
     </inertial>
     <visual>
-      <origin rpy="0 0 0" xyz="0.008 0.65425 -0.8115"/>
-      <geometry>
-        <mesh filename="package://arm_22_gazebo_pos/meshes/parmak_1_link_1.stl" scale="0.001 0.001 0.001"/>
-      </geometry>
-      <material name="silver"/>
-    </visual>
-    <collision>
-      <origin rpy="0 0 0" xyz="0.008 0.65425 -0.8115"/>
-      <geometry>
-        <mesh filename="package://arm_22_gazebo_pos/meshes/parmak_1_link_1.stl" scale="0.001 0.001 0.001"/>
+      <origin rpy="0 0 0" xyz="0.008 0.5025 -0.8115"/>
+      <geometry>
+        <mesh filename="package://arm_22_gazebo_pos_65_67/meshes/parmak_1_link_1.stl" scale="0.001 0.001 0.001"/>
+      </geometry>
+      <material name="silver"/>
+    </visual>
+    <collision>
+      <origin rpy="0 0 0" xyz="0.008 0.5025 -0.8115"/>
+      <geometry>
+        <mesh filename="package://arm_22_gazebo_pos_65_67/meshes/parmak_1_link_1.stl" scale="0.001 0.001 0.001"/>
       </geometry>
     </collision>
@@ -178,14 +184,14 @@
     </inertial>
     <visual>
-      <origin rpy="0 0 0" xyz="-0.008 0.65425 -0.8115"/>
-      <geometry>
-        <mesh filename="package://arm_22_gazebo_pos/meshes/parmak_2_link_1.stl" scale="0.001 0.001 0.001"/>
-      </geometry>
-      <material name="silver"/>
-    </visual>
-    <collision>
-      <origin rpy="0 0 0" xyz="-0.008 0.65425 -0.8115"/>
-      <geometry>
-        <mesh filename="package://arm_22_gazebo_pos/meshes/parmak_2_link_1.stl" scale="0.001 0.001 0.001"/>
+      <origin rpy="0 0 0" xyz="-0.008 0.50425 -0.8115"/>
+      <geometry>
+        <mesh filename="package://arm_22_gazebo_pos_65_67/meshes/parmak_2_link_1.stl" scale="0.001 0.001 0.001"/>
+      </geometry>
+      <material name="silver"/>
+    </visual>
+    <collision>
+      <origin rpy="0 0 0" xyz="-0.008 0.50425 -0.8115"/>
+      <geometry>
+        <mesh filename="package://arm_22_gazebo_pos_65_67/meshes/parmak_2_link_1.stl" scale="0.001 0.001 0.001"/>
       </geometry>
     </collision>

Commit message: #51 New link lenghts fixed.

File: rover_22_robotic_arm/new_links/arm_22_gazebo_pos_50_55/urdf/assembly.urdf.xacro (robot description, xacro)
@@ -144,5 +144,5 @@
     </inertial>
     <visual>
-      <origin rpy="0 0 0" xyz="-0.0 0.40925 -0.8965"/>
+      <origin rpy="0 0 0" xyz="-0.0 0.5725 -0.8965"/>
       <geometry>
         <mesh filename="package://arm_22_gazebo_pos_50_55/meshes/gripper_link_1.stl" scale="0.001 0.001 0.001"/>
@@ -226,5 +226,5 @@
   </joint>
   <joint name="axis_5" type="continuous">
-    <origin rpy="0 0 0" xyz="0.055 -0.398 0.0"/>
+    <origin rpy="0 0 0" xyz="-0.025 -0.398 0.0"/>
     <parent link="4_5_link_1"/>
     <child link="5_6_link_1"/>
@@ -233,5 +233,5 @@
   </joint>
   <joint name="axis_6" type="continuous">
-    <origin rpy="0 0 0" xyz="-0.055 -0.022 0.0"/>
+    <origin rpy="0 0 0" xyz="-0.000 -0.022 0.0"/>
     <parent link="5_6_link_1"/>
     <child link="gripper_link_1"/>

File: rover_22_robotic_arm/new_links/arm_22_gazebo_pos_55_50/urdf/assembly.urdf.xacro (robot description, xacro)
@@ -144,5 +144,5 @@
     </inertial>
     <visual>
-      <origin rpy="0 0 0" xyz="-0.0 0.40925 -0.8965"/>
+      <origin rpy="0 0 0" xyz="-0.0 0.5725 -0.8965"/>
       <geometry>
         <mesh filename="package://arm_22_gazebo_pos_55_50/meshes/gripper_link_1.stl" scale="0.001 0.001 0.001"/>
@@ -219,5 +219,5 @@
   </joint>
   <joint name="axis_4" type="continuous">
-    <origin rpy="0 0 0" xyz="0.025 -0.14925 0.0"/>
+    <origin rpy="0 0 0" xyz="0.025 -0.22925 0.0"/>
     <parent link="3_4_link_1"/>
     <child link="4_5_link_1"/>
@@ -226,5 +226,5 @@
   </joint>
   <joint name="axis_5" type="continuous">
-    <origin rpy="0 0 0" xyz="0.055 -0.398 0.0"/>
+    <origin rpy="0 0 0" xyz="-0.025 -0.318 0.0"/>
     <parent link="4_5_link_1"/>
     <child link="5_6_link_1"/>
@@ -233,5 +233,5 @@
   </joint>
   <joint name="axis_6" type="continuous">
-    <origin rpy="0 0 0" xyz="-0.055 -0.022 0.0"/>
+    <origin rpy="0 0 0" xyz="-0.0 -0.192 0.0"/>
     <parent link="5_6_link_1"/>
     <child link="gripper_link_1"/>

File: rover_22_robotic_arm/new_links/arm_22_gazebo_pos_55_55/urdf/assembly.urdf.xacro (robot description, xacro)
@@ -124,5 +124,5 @@
     </inertial>
     <visual>
-      <origin rpy="0 0 0" xyz="-0.055 0.44725 -0.8965"/>
+      <origin rpy="0 0 0" xyz="-0.055 0.47725 -0.8965"/>
       <geometry>
         <mesh filename="package://arm_22_gazebo_pos_55_55/meshes/5_6_link_1.stl" scale="0.001 0.001 0.001"/>
@@ -144,5 +144,5 @@
     </inertial>
     <visual>
-      <origin rpy="0 0 0" xyz="-0.0 0.40925 -0.8965"/>
+      <origin rpy="0 0 0" xyz="-0.0 0.47925 -0.8965"/>
       <geometry>
         <mesh filename="package://arm_22_gazebo_pos_55_55/meshes/gripper_link_1.stl" scale="0.001 0.001 0.001"/>
@@ -212,5 +212,5 @@
   </joint>
   <joint name="axis_3" type="continuous">
-    <origin rpy="0 0 0" xyz="-0.0465 0.0 0.6555"/>
+    <origin rpy="0 0 0" xyz="-0.0465 0.0 0.555"/>
     <parent link="2_3_link_1"/>
     <child link="3_4_link_1"/>
@@ -219,5 +219,5 @@
   </joint>
   <joint name="axis_4" type="continuous">
-    <origin rpy="0 0 0" xyz="0.025 -0.14925 0.0"/>
+    <origin rpy="0 0 0" xyz="0.025 -0.2925 0.0"/>
     <parent link="3_4_link_1"/>
     <child link="4_5_link_1"/>
@@ -226,5 +226,5 @@
   </joint>
   <joint name="axis_5" type="continuous">
-    <origin rpy="0 0 0" xyz="0.055 -0.398 0.0"/>
+    <origin rpy="0 0 0" xyz="-0.025 -0.398 0.0"/>
     <parent link="4_5_link_1"/>
     <child link="5_6_link_1"/>
@@ -233,5 +233,5 @@
   </joint>
   <joint name="axis_6" type="continuous">
-    <origin rpy="0 0 0" xyz="-0.055 -0.022 0.0"/>
+    <origin rpy="0 0 0" xyz="0.0 -0.022 0.0"/>
     <parent link="5_6_link_1"/>
     <child link="gripper_link_1"/>
