Commit message: Fix joint positions in urdf

File: rover_22_robotic_arm/new_links/arm_22_gazebo_pos_55_55/urdf/assembly.urdf.xacro (robot description, xacro)
@@ -205,5 +205,5 @@
   </joint>
   <joint name="axis_2" type="continuous">
-    <origin rpy="0 0 0" xyz="0.0215 0.0 0.0875"/>
+    <origin rpy="0 0 0" xyz="0.0 0.0 0.0875"/>
     <parent link="1_2_link_1"/>
     <child link="2_3_link_1"/>
@@ -212,5 +212,5 @@
   </joint>
   <joint name="axis_3" type="continuous">
-    <origin rpy="0 0 0" xyz="-0.0465 0.0 0.555"/>
+    <origin rpy="0 0 0" xyz="0.0 0.0 0.550"/>
     <parent link="2_3_link_1"/>
     <child link="3_4_link_1"/>
@@ -219,5 +219,5 @@
   </joint>
   <joint name="axis_4" type="continuous">
-    <origin rpy="0 0 0" xyz="0.025 -0.2925 0.0"/>
+    <origin rpy="0 0 0" xyz="0.0 -0.22 0.0"/>
     <parent link="3_4_link_1"/>
     <child link="4_5_link_1"/>
@@ -226,5 +226,5 @@
   </joint>
   <joint name="axis_5" type="continuous">
-    <origin rpy="0 0 0" xyz="-0.025 -0.398 0.0"/>
+    <origin rpy="0 0 0" xyz="-0.0 -0.28 0.0"/>
     <parent link="4_5_link_1"/>
     <child link="5_6_link_1"/>

Commit message: Fix 55-55 lenght.

File: rover_22_robotic_arm/new_links/arm_22_gazebo_pos_55_55/urdf/assembly.urdf.xacro (robot description, xacro)
@@ -80,5 +80,5 @@
     </inertial>
     <visual>
-      <origin rpy="0 0 0" xyz="0.025 -0.14 -0.1"/>
+      <origin rpy="0 0 0" xyz="0.0 -0.14 0.0"/>
       <geometry>
         <!-- <mesh filename="package://arm_22_gazebo_pos_55_55/meshes/3_4_link_1.stl" scale="0.001 0.001 0.001"/> -->
@@ -88,5 +88,5 @@
     </visual>
     <collision>
-      <origin rpy="0 0 0" xyz="0.025 -0.14 -0.1"/>
+      <origin rpy="0 0 0" xyz="0.0 -0.14 0.0"/>
       <geometry>
         <!-- <mesh filename="package://arm_22_gazebo_pos_55_55/meshes/3_4_link_1.stl" scale="0.001 0.001 0.001"/> -->
@@ -102,16 +102,16 @@
     </inertial>
     <visual>
-      <origin rpy="0 0 0" xyz="-0.0 -0.28325 -0.1"/>
+      <origin rpy="0 0 0" xyz="-0.0 -0.18325 0.0"/>
       <geometry>
         <!-- <mesh filename="package://arm_22_gazebo_pos_55_55/meshes/4_5_link_1.stl" scale="0.001 0.001 0.001"/> -->
-        <box size="0.05 0.275 0.05" />
-      </geometry>
-      <material name="silver"/>
-    </visual>
-    <collision>
-      <origin rpy="0 0 0" xyz="-0.0 -0.283925 -0.1"/>
+        <box size="0.05 0.375 0.05" />
+      </geometry>
+      <material name="silver"/>
+    </visual>
+    <collision>
+      <origin rpy="0 0 0" xyz="-0.0 -0.183925 0.0"/>
       <geometry>
         <!-- <mesh filename="package://arm_22_gazebo_pos_55_55/meshes/4_5_link_1.stl" scale="0.001 0.001 0.001"/> -->
-        <box size="0.05 0.275 0.05" />
+        <box size="0.05 0.375 0.05" />
       </geometry>
     </collision>
@@ -124,5 +124,5 @@
     </inertial>
     <visual>
-      <origin rpy="0 0 0" xyz="-0.055 0.47725 -0.8965"/>
+      <origin rpy="0 0 0" xyz="-0.055 0.47725 -0.7965"/>
       <geometry>
         <mesh filename="package://arm_22_gazebo_pos_55_55/meshes/5_6_link_1.stl" scale="0.001 0.001 0.001"/>
@@ -131,5 +131,5 @@
     </visual>
     <collision>
-      <origin rpy="0 0 0" xyz="-0.055 0.44725 -0.8965"/>
+      <origin rpy="0 0 0" xyz="-0.055 0.44725 -0.7965"/>
       <geometry>
         <mesh filename="package://arm_22_gazebo_pos_55_55/meshes/5_6_link_1.stl" scale="0.001 0.001 0.001"/>
@@ -144,5 +144,5 @@
     </inertial>
     <visual>
-      <origin rpy="0 0 0" xyz="-0.0 0.47925 -0.8965"/>
+      <origin rpy="0 0 0" xyz="-0.0 0.47925 -0.7965"/>
       <geometry>
         <mesh filename="package://arm_22_gazebo_pos_55_55/meshes/gripper_link_1.stl" scale="0.001 0.001 0.001"/>
@@ -151,5 +151,5 @@
     </visual>
     <collision>
-      <origin rpy="0 0 0" xyz="-0.0 0.40925 -0.8965"/>
+      <origin rpy="0 0 0" xyz="-0.0 0.40925 -0.7965"/>
       <geometry>
         <mesh filename="package://arm_22_gazebo_pos_55_55/meshes/gripper_link_1.stl" scale="0.001 0.001 0.001"/>
@@ -164,5 +164,5 @@
     </inertial>
     <visual>
-      <origin rpy="0 0 0" xyz="0.008 0.4925 -0.9115"/>
+      <origin rpy="0 0 0" xyz="0.008 0.5925 -0.8115"/>
       <geometry>
         <mesh filename="package://arm_22_gazebo_pos_55_55/meshes/parmak_1_link_1.stl" scale="0.001 0.001 0.001"/>
@@ -171,5 +171,5 @@
     </visual>
     <collision>
-      <origin rpy="0 0 0" xyz="0.008 0.4925 -0.9115"/>
+      <origin rpy="0 0 0" xyz="0.008 0.5925 -0.8115"/>
       <geometry>
         <mesh filename="package://arm_22_gazebo_pos_55_55/meshes/parmak_1_link_1.stl" scale="0.001 0.001 0.001"/>
@@ -184,5 +184,5 @@
     </inertial>
     <visual>
-      <origin rpy="0 0 0" xyz="-0.008 0.49425 -0.9115"/>
+      <origin rpy="0 0 0" xyz="-0.008 0.59425 -0.8115"/>
       <geometry>
         <mesh filename="package://arm_22_gazebo_pos_55_55/meshes/parmak_2_link_1.stl" scale="0.001 0.001 0.001"/>
@@ -191,5 +191,5 @@
     </visual>
     <collision>
-      <origin rpy="0 0 0" xyz="-0.008 0.49425 -0.9115"/>
+      <origin rpy="0 0 0" xyz="-0.008 0.59425 -0.8115"/>
       <geometry>
         <mesh filename="package://arm_22_gazebo_pos_55_55/meshes/parmak_2_link_1.stl" scale="0.001 0.001 0.001"/>
@@ -205,5 +205,5 @@
   </joint>
   <joint name="axis_2" type="continuous">
-    <origin rpy="0 0 0" xyz="0.0215 0.0 0.0875"/>
+    <origin rpy="0 0 0" xyz="0.0 0.0 0.0875"/>
     <parent link="1_2_link_1"/>
     <child link="2_3_link_1"/>
@@ -212,5 +212,5 @@
   </joint>
   <joint name="axis_3" type="continuous">
-    <origin rpy="0 0 0" xyz="-0.0465 0.0 0.555"/>
+    <origin rpy="0 0 0" xyz="0.0 0.0 0.550"/>
     <parent link="2_3_link_1"/>
     <child link="3_4_link_1"/>
@@ -219,5 +219,5 @@
   </joint>
   <joint name="axis_4" type="continuous">
-    <origin rpy="0 0 0" xyz="0.025 -0.2925 0.0"/>
+    <origin rpy="0 0 0" xyz="0.0 -0.22 0.0"/>
     <parent link="3_4_link_1"/>
     <child link="4_5_link_1"/>
@@ -226,5 +226,5 @@
   </joint>
   <joint name="axis_5" type="continuous">
-    <origin rpy="0 0 0" xyz="-0.025 -0.398 0.0"/>
+    <origin rpy="0 0 0" xyz="-0.0 -0.28 0.0"/>
     <parent link="4_5_link_1"/>
     <child link="5_6_link_1"/>

Commit message: #54 Lneght fixed and end effector added.

File: rover_22_robotic_arm/new_links/arm_22_gazebo_pos_55_55/urdf/assembly.urdf.xacro (robot description, xacro)
@@ -197,4 +197,6 @@
     </collision>
   </link>
+  <link name="end_effector">
+  </link>
   <joint name="axis_1" type="continuous">
     <origin rpy="0 0 0" xyz="0.0 0.0 0.0535"/>
@@ -253,3 +255,8 @@
     <limit lower="-0.05" upper="0.5" effort="200" velocity="20" />
   </joint>
+  <joint name="center_gripper" type="fixed">
+    <origin rpy="0 0 0" xyz="0.0 -0.238 0.0"/>
+    <parent link="gripper_link_1"/>
+    <child link="end_effector"/>
+  </joint>
 </robot>

Commit message: #55 Collisons fixed.

File: rover_22_robotic_arm/new_links/arm_22_gazebo_pos_55_55/urdf/assembly.urdf.xacro (robot description, xacro)
@@ -131,5 +131,5 @@
     </visual>
     <collision>
-      <origin rpy="0 0 0" xyz="-0.055 0.44725 -0.7965"/>
+      <origin rpy="0 0 0" xyz="-0.055 0.47725 -0.7965"/>
       <geometry>
         <mesh filename="package://arm_22_gazebo_pos_55_55/meshes/5_6_link_1.stl" scale="0.001 0.001 0.001"/>
@@ -151,5 +151,5 @@
     </visual>
     <collision>
-      <origin rpy="0 0 0" xyz="-0.0 0.40925 -0.7965"/>
+      <origin rpy="0 0 0" xyz="-0.0 0.47925 -0.7965"/>
       <geometry>
         <mesh filename="package://arm_22_gazebo_pos_55_55/meshes/gripper_link_1.stl" scale="0.001 0.001 0.001"/>
